File: NPN Tracer/NPN Tracer V1/NPN Tracer V1.kicad_pcb (KiCad board)
At the start: 2 copper layers, 89.9 x 69.9 mm, 48 parts, among them J1 AD3, J2 AD4, J3 AD2, J4 RCSEL, J5 PWR, J6 AD1, J7 +5, J8 13.8V MAX, Q1 TIP120, U1 LM358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

Commit message: Update 8May23
Parts:
- ADC1, ADC2, ADC3, ADC4: value 10K -> 100K
Changed lines of the file:
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@@
       (effects (font (size 1 1) (thickness 0.15)))
     )
-    (fp_text value "10K" (at 3.2875 -0.0245) (layer "F.SilkS")
+    (fp_text value "100K" (at 3.2875 -0.0245) (layer "F.SilkS")
       (effects (font (size 1 1) (thickness 0.15)))
     )
@@
       (effects (font (size 1 1) (thickness 0.15)))
     )
-    (fp_text value "10K" (at 1.0695 3.4925 -90) (layer "F.SilkS")
+    (fp_text value "100K" (at 1.0695 3.4925 -90) (layer "F.SilkS")
       (effects (font (size 1 1) (thickness 0.15)))
     )
@@
     (property "Sheetname" "")
     (attr through_hole)
-    (fp_text reference "TB1" (at -6.8825 20.3345 180) (layer "F.SilkS")
+    (fp_text reference "TB1" (at -4.755 -22.789 180) (layer "F.SilkS")
       (effects (font (size 1.4 1.4) (thickness 0.15)))
     )
-    (fp_text value "NANO" (at 6.0715 20.525 180) (layer "F.SilkS")
+    (fp_text value "NANO" (at 7.591 27.891 180) (layer "F.Fab")
       (effects (font (size 1.4 1.4) (thickness 0.15)))
     )
     (fp_line (start -8.89 21.59) (end -8.89 -21.59) (layer "F.SilkS") (width 0.127))
+    (fp_line (start 8.89 21.59) (end -8.89 21.59) (layer "F.SilkS") (width 0.127))
     (fp_line (start 8.89 -21.59) (end 8.89 21.59) (layer "F.SilkS") (width 0.127))
-    (fp_line (start 8.89 21.59) (end -8.89 21.59) (layer "F.SilkS") (width 0.127))
     (fp_line (start -8.89 -21.59) (end 8.89 -21.59) (layer "F.SilkS") (width 0.127))
     (fp_circle (center -10.2 -17.8) (end -10.1 -17.8) (layer "F.SilkS") (width 0.2) (fill none))
-    (fp_line (start -9.14 21.84) (end -3.22 21.84) (layer "F.CrtYd") (width 0.05))
-    (fp_line (start 9.14 -21.84) (end 9.14 21.84) (layer "F.CrtYd") (width 0.05))
-    (fp_line (start -9.14 21.84) (end -9.14 -21.84) (layer "F.CrtYd") (width 0.05))
-    (fp_line (start -3.22 21.84) (end -3.22 23.745) (layer "F.CrtYd") (width 0.05))
     (fp_line (start -9.14 -21.84) (end 9.14 -21.84) (layer "F.CrtYd") (width 0.05))
     (fp_line (start -3.22 23.745) (end 3.25 23.745) (layer "F.CrtYd") (width 0.05))
     (fp_line (start 3.25 21.84) (end 9.14 21.84) (layer "F.CrtYd") (width 0.05))
+    (fp_line (start 9.14 -21.84) (end 9.14 21.84) (layer "F.CrtYd") (width 0.05))
+    (fp_line (start -3.22 21.84) (end -3.22 23.745) (layer "F.CrtYd") (width 0.05))
+    (fp_line (start -9.14 21.84) (end -9.14 -21.84) (layer "F.CrtYd") (width 0.05))
+    (fp_line (start -9.14 21.84) (end -3.22 21.84) (layer "F.CrtYd") (width 0.05))
     (fp_line (start 3.25 23.745) (end 3.25 21.84) (layer "F.CrtYd") (width 0.05))
-    (fp_line (start -8.89 -21.59) (end 8.89 -21.59) (layer "F.Fab") (width 0.127))
+    (fp_line (start -2.97 23.495) (end 3 23.495) (layer "F.Fab") (width 0.127))
     (fp_line (start -2.97 21.59) (end -8.89 21.59) (layer "F.Fab") (width 0.127))
+    (fp_line (start 8.89 -21.59) (end 8.89 21.59) (layer "F.Fab") (width 0.127))
+    (fp_line (start 3 23.495) (end 3 21.59) (layer "F.Fab") (width 0.127))
     (fp_line (start -2.97 21.59) (end -2.97 23.495) (layer "F.Fab") (width 0.127))
     (fp_line (start -8.89 21.59) (end -8.89 -21.59) (layer "F.Fab") (width 0.127))
-    (fp_line (start 8.89 -21.59) (end 8.89 21.59) (layer "F.Fab") (width 0.127))
+    (fp_line (start -8.89 -21.59) (end 8.89 -21.59) (layer "F.Fab") (width 0.127))
     (fp_line (start 8.89 21.59) (end 3 21.59) (layer "F.Fab") (width 0.127))
     (fp_line (start 3 21.59) (end -2.97 21.59) (layer "F.Fab") (width 0.127))
-    (fp_line (start -2.97 23.495) (end 3 23.495) (layer "F.Fab") (width 0.127))
-    (fp_line (start 3 23.495) (end 3 21.59) (layer "F.Fab") (width 0.127))
     (fp_circle (center -10.2 -17.8) (end -10.1 -17.8) (layer "F.Fab") (width 0.2) (fill none))
     (pad "1" thru_hole rect (at -7.62 -17.78 180) (size 1.8 1.8) (drill 0.9) (layers *.Cu *.Mask)
@@
       (effects (font (size 1 1) (thickness 0.15)))
     )
-    (fp_text value "10K" (at -4.914 3.6585 -90) (layer "F.SilkS")
+    (fp_text value "100K" (at -4.914 3.6585 -90) (layer "F.SilkS")
       (effects (font (size 1 1) (thickness 0.15)))
     )
@@
     (property "Sheetname" "")
     (attr through_hole)
-    (fp_text reference "R3" (at 5.3475 3.1115 180) (layer "F.SilkS")
-      (effects (font (size 1 1) (thickness 0.15)))
-    )
-    (fp_text value "200" (at 4.776 1.778) (layer "F.SilkS")
+    (fp_text reference "R3" (at 4.6165 3.1255 180) (layer "F.SilkS")
+      (effects (font (size 1 1) (thickness 0.15)))
+    )
+    (fp_text value "200" (at 4.0765 1.7955) (layer "F.SilkS")
       (effects (font (size 1 1) (thickness 0.15)))
     )
@@
       (effects (font (size 1 1) (thickness 0.15)))
     )
-    (fp_text value "10K" (at 1.133 3.4925 -90) (layer "F.SilkS")
-      (effects (font (size 1 1) (thickness 0.15)))
-    )
+    (fp_text value "100K" (at 1.133 3.4925 -90) (layer "F.SilkS")
+      (effects (font (size 1 1) (thickness 0.15)))
+    )
