File: NPN Tracer/NPN Tracer V1/NPN Tracer V1.kicad_sch (KiCad schematic)
At the start: 48 parts, among them J1 AD3, J2 AD4, J3 AD2, J4 RCSEL, J5 PWR, J6 AD1, J7 +5, J8 13.8V MAX, Q1 TIP120, U1 LM358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

Commit message: Update 8May23
Parts:
- C5: value 22u -> 1u
- R11, R4: value 500 -> 499
Other:
- moved on the sheet: C10, C7, C8, C9, D1, D3, D4, D5, D6, J5, J8
